File: Eigene Steuerplatine Line Decoder.kicad_pcb (KiCad board)
At the start: 2 copper layers, 100 x 100 mm, 32 parts, among them P1 POWER/DATA, P2 LED, P3 MATRIX, P4 MUX, Q1 BC547, Q2 IRF740, U1 R-78E5.0-0.5, U2 LM317T, U3 CD4514B, U4 ULN2803A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

Commit message: Convert to KiCad 7 project
Other:
- net class Default removed
- net class Power removed
